File: PI4Adapter.kicad_pcb (KiCad board)
At the start: 2 copper layers, 39.3 x 56.3 mm, 5 parts, among them J1 Conn_02x20_Odd_Even, J2 Conn_02x20_Odd_Even, J3 Conn_02x13_Odd_Even, J4 Conn_01x02_Male, U1 USB_C_2.0

Commit message: update
Routing:
- net +5V: track 127.8 -> 87.0 mm, vias 15 -> 0
- net GND: track 100.6 -> 82.0 mm, vias 15 -> 2
- net GPIO27: track 32.8 -> 35.7 mm
- net GPIO23: track 32.4 -> 34.7 mm
- net GPIO25: track 32.8 -> 35.0 mm
- net GPIO22: track 36.1 -> 34.3 mm
- net GPIO10: track 34.8 -> 33.2 mm
- net GPIO8: track 32.4 -> 33.9 mm
- net GPIO3: track 34.0 -> 32.9 mm
- net GPIO9: track 33.1 -> 34.1 mm
- net GPIO17: track 33.9 -> 32.9 mm
- net GPIO7: track 32.8 -> 33.7 mm
- net GPIO18: track 34.1 -> 33.3 mm
- net GPIO6: track 11.2 -> 11.9 mm
- net GPIO24: track 33.4 -> 32.8 mm
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Other:
- board text added: "PI Duet 3 Adapter v0.1b"
- board text removed: "PI3/PI4 Duet 3 Adapter v0.1a"

Commit message: update
Parts:
- removed U1: USB_C_2.0, Library:USB_C_C31M17
- added J5: USB_C_Receptacle_PowerOnly_6P, Connector_USB:USB_C_Receptacle_GCT_USB4135-GF-A_6P_TopMnt_Horizontal, F.Cu at (128.9, 126.4)
- moved J2 3.46 mm to (115.6, 77.6)
- moved J4 1.98 mm to (129.5, 83.0)
Routing:
- net GND: track 82.0 -> 144.1 mm, vias 2 -> 0
- net IDSD: track 11.9 -> 8.49 mm
- net GPIO19: track 12.0 -> 8.55 mm
- net GPIO6: track 11.9 -> 8.54 mm
- net GPIO13: track 11.9 -> 8.55 mm
- net GPIO26: track 11.9 -> 8.55 mm
- net GPIO5: track 11.9 -> 8.56 mm
- net GPIO16: track 11.8 -> 8.49 mm
- net GPIO21: track 11.8 -> 8.55 mm
- net IDSC: track 11.7 -> 8.49 mm
- net GPIO12: track 11.7 -> 8.50 mm
- net GPIO20: track 11.7 -> 8.55 mm
- net +3.3V: track 87.8 -> 85.2 mm
- net GPIO3: track 32.9 -> 35.5 mm
- net GPIO27: track 35.7 -> 33.2 mm
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- removed copper zone on B.Cu, net GND
Other:
- board size 39.3 x 56.3 mm -> 39.7 x 56.3 mm
- board text added: "locked"
- board text removed: "+"
- board text removed: "5vdc"
- board text removed: "CC BY-SA 4.0"
- board text removed: "PI Duet 3 Adapter v0.1b"
- board text removed: "USB C Power"
